File: teatime.sch (KiCad schematic (older format))
At the start: 64 parts, among them Q1 NCV8402, Q2 NCV8402, Q3 NCV8402, Q4 NCV8402, Q5 NCV8402, Q6 NCV8402, Q7 NCV8402, Q8 NCV8402, SW1 SW_Push, U1 NCP1117-3.3_SOT223, U2 74HC4051

Commit message: Shift regs and led layout
Parts:
- removed BT2: Battery_Cell, Battery:BatteryHolder_Keystone_1058_1x2032, symbol Device:Battery_Cell
- removed Q1, Q2, Q3, Q4, Q5, Q6, Q7, Q8: NCV8402, Package_TO_SOT_SMD:SOT-223-3_TabPin2, symbol Device:Q_NMOS_GDS
- removed SW1: SW_Push, Button_Switch_THT:SW_PUSH-12mm, symbol Switch:SW_Push
- removed U2: 74HC4051, Package_SO:SOP-16_4.4x10.4mm_P1.27mm, symbol 74xx:74HC4051
- added D25, D26, D27, D28, D29, D30, D31, D32: LED, LED_THT:LED_D5.0mm, symbol Device:LED_Small
- added H1, H2, H3, H4: MountingHole, MountingHole:MountingHole_3.2mm_M3, symbol Mechanical:MountingHole
- added R26, R27, R28, R29, R30, R31, R32: 680r, Resistor_THT:R_Axial_DIN0204_L3.6mm_D1.6mm_P5.08mm_Horizontal, symbol Device:R_Small
- added U2, U3, U4, U5: 74HC596, Package_DIP:DIP-16_W7.62mm, symbol 74xx:74HC596
- BT1: footprint Battery:BatteryHolder_Keystone_1058_1x2032 -> Connector_JST:JST_PH_S2B-PH-K_1x02_P2.00mm_Horizontal
- D1, D10, D11, D12, D13, D14, D15, D16, D17, D18, D19, D2, D20, D21, D22, D23, D24, D3, D4, D5, D6, D7, D8, D9: footprint LED_THT:LED_D5.0mm_Clear -> LED_THT:LED_D5.0mm
- R1, R12, R13, R18, R19, R2, R24, R25, R7: value R_Small -> 680r; footprint Resistor_SMD:R_1206_3216Metric -> Resistor_THT:R_Axial_DIN0204_L3.6mm_D1.6mm_P5.08mm_Horizontal
- R10, R11, R16, R17, R22, R23, R5, R6: value 100k -> 680r; footprint Resistor_SMD:R_1206_3216Metric -> Resistor_THT:R_Axial_DIN0204_L3.6mm_D1.6mm_P5.08mm_Horizontal
- R14, R15, R20, R21, R3, R4, R8, R9: value 1k -> 680r; footprint Resistor_SMD:R_1206_3216Metric -> Resistor_THT:R_Axial_DIN0204_L3.6mm_D1.6mm_P5.08mm_Horizontal
Connections:
- net labels added: +3V3
- net labels removed: VCC
- wire segments 94 -> 145
- no-connect marks 0 -> 1
Other:
- moved on the sheet: BT1, C1, C2

Commit message: Add micro and tweak some other bits
Parts:
- removed U1: NCP1117-3.3_SOT223, Package_TO_SOT_SMD:SOT-223-3_TabPin2, symbol Regulator_Linear:NCP1117-3.3_SOT223
- added R33: 100k, Resistor_THT:R_Axial_DIN0204_L3.6mm_D1.6mm_P5.08mm_Horizontal, symbol Device:R_Small
- added SW1: SW_Push, Button_Switch_THT:SW_PUSH_6mm, symbol Switch:SW_Push
- added U1: MCP1700-3302E_TO92, Package_TO_SOT_THT:TO-92_Inline, symbol Regulator_Linear:MCP1700-3302E_TO92
- added U6: ATtiny85-20PU, Package_DIP:DIP-8_W7.62mm, symbol MCU_Microchip_ATtiny:ATtiny85-20PU
- R1, R10, R11, R12, R13, R14, R15, R16, R17, R18, R19, R2, R20, R21, R22, R23, R24, R25, R26, R27, R28, R29, R3, R30, R31, R32, R4, R5, R6, R7, R8, R9: value 680r -> 220r
Connections:
- wire segments 145 -> 148
- no-connect marks 1 -> 3
Other:
- moved on the sheet: D1, D10, D11, D12, D13, D14, D15, D16, D17, D18, D19, D2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

Commit message: More tweaks and v1 version of board
Parts:
- added C3: 100n, Capacitor_THT:C_Disc_D3.0mm_W1.6mm_P2.50mm, symbol Device:C_Small
- C1, C2: value 10u -> 1u
Connections:
- wire segments 148 -> 150
Changed lines of the file:
@@
 EESchema Schematic File Version 4
-EELAYER 30 0
+LIBS:teatime-cache
+EELAYER 26 0
 EELAYER END
 $Descr A4 11693 8268
@@
 P 1700 1000
 F 0 "C1" H 1792 1046 50  0000 L CNN
-F 1 "10u" H 1792 955 50  0000 L CNN
+F 1 "1u" H 1792 955 50  0000 L CNN
 F 2 "Capacitor_SMD:C_1206_3216Metric" H 1700 1000 50  0001 C CNN
 F 3 "~" H 1700 1000 50  0001 C CNN
@@
 P 2700 1000
 F 0 "C2" H 2792 1046 50  0000 L CNN
-F 1 "10u" H 2792 955 50  0000 L CNN
+F 1 "1u" H 2792 955 50  0000 L CNN
 F 2 "Capacitor_SMD:C_1206_3216Metric" H 2700 1000 50  0001 C CNN
 F 3 "~" H 2700 1000 50  0001 C CNN
@@
 L power:+3V3 #PWR014
 U 1 1 5E4A3888
-P 2700 2000
-F 0 "#PWR014" H 2700 1850 50  0001 C CNN
-F 1 "+3V3" H 2715 2173 50  0000 C CNN
-F 2 "" H 2700 2000 50  0001 C CNN
-F 3 "" H 2700 2000 50  0001 C CNN
-	1    2700 2000
+P 2700 1700
+F 0 "#PWR014" H 2700 1550 50  0001 C CNN
+F 1 "+3V3" H 2715 1873 50  0000 C CNN
+F 2 "" H 2700 1700 50  0001 C CNN
+F 3 "" H 2700 1700 50  0001 C CNN
+	1    2700 1700
 	1    0    0    -1
 $EndComp
@@
 	-1   0    0    1
 $EndComp
+$Comp
+L Device:C_Small C3
+U 1 1 5E44F96C
+P 2350 1800
+F 0 "C3" H 2442 1846 50  0000 L CNN
+F 1 "100n" H 2442 1755 50  0000 L CNN
+F 2 "Capacitor_THT:C_Disc_D3.0mm_W1.6mm_P2.50mm" H 2350 1800 50  0001 C CNN
+F 3 "~" H 2350 1800 50  0001 C CNN
+	1    2350 1800
+	1    0    0    -1
+$EndComp
+$Comp
+L power:GND #PWR018
+U 1 1 5E44FA46
+P 2350 1900
+F 0 "#PWR018" H 2350 1650 50  0001 C CNN
+F 1 "GND" H 2355 1727 50  0000 C CNN
+F 2 "" H 2350 1900 50  0001 C CNN
+F 3 "" H 2350 1900 50  0001 C CNN
+	1    2350 1900
+	1    0    0    -1
+$EndComp
+Wire Wire Line
+	2350 1700 2700 1700
+Wire Wire Line
+	2700 1700 2700 2000
+Connection ~ 2700 1700
 $EndSCHEMATC

Commit message: Few slight tweaks to footprints used and updated build files
Parts:
- C3: footprint Capacitor_THT:C_Disc_D3.0mm_W1.6mm_P2.50mm -> Capacitor_SMD:C_1206_3216Metric
- U1: footprint Package_TO_SOT_THT:TO-92_Inline -> Package_TO_SOT_THT:TO-92_Inline_W4.0mm_Horizontal_FlatSideDown
- U2, U3, U4, U5: value 74HC596 -> 74HC595; symbol 74xx:74HC596 -> 74xx:74HC595
Changed lines of the file:
@@
 	1700 900  700  900
 $Comp
-L 74xx:74HC596 U2
+L 74xx:74HC595 U2
 U 1 1 5E43099D
 P 5450 1950
 F 0 "U2" V 5450 1950 50  0000 C CNN
-F 1 "74HC596" V 5550 1950 50  0000 C CNN
+F 1 "74HC595" V 5550 1950 50  0000 C CNN
 F 2 "Package_DIP:DIP-16_W7.62mm" H 5450 1950 50  0001 C CNN
 F 3 "https://assets.nexperia.com/documents/data-sheet/74HC_HCT595.pdf" H 5450 1950 50  0001 C CNN
@@
 Connection ~ 5450 2650
 $Comp
-L 74xx:74HC596 U3
+L 74xx:74HC595 U3
 U 1 1 5E44C9F4
 P 6250 3150
 F 0 "U3" V 6250 3150 50  0000 C CNN
-F 1 "74HC596" V 6350 3150 50  0000 C CNN
+F 1 "74HC595" V 6350 3150 50  0000 C CNN
 F 2 "Package_DIP:DIP-16_W7.62mm" H 6250 3150 50  0001 C CNN
 F 3 "https://assets.nexperia.com/documents/data-sheet/74HC_HCT595.pdf" H 6250 3150 50  0001 C CNN
@@
 Connection ~ 6250 3850
 $Comp
-L 74xx:74HC596 U4
+L 74xx:74HC595 U4
 U 1 1 5E44CAA4
 P 7050 4350
 F 0 "U4" V 7050 4350 50  0000 C CNN
-F 1 "74HC596" V 7150 4350 50  0000 C CNN
+F 1 "74HC595" V 7150 4350 50  0000 C CNN
 F 2 "Package_DIP:DIP-16_W7.62mm" H 7050 4350 50  0001 C CNN
 F 3 "https://assets.nexperia.com/documents/data-sheet/74HC_HCT595.pdf" H 7050 4350 50  0001 C CNN
@@
 Connection ~ 7050 5050
 $Comp
-L 74xx:74HC596 U5
+L 74xx:74HC595 U5
 U 1 1 5E44CB56
 P 7850 5550
 F 0 "U5" V 7850 5550 50  0000 C CNN
-F 1 "74HC596" V 7950 5550 50  0000 C CNN
+F 1 "74HC595" V 7950 5550 50  0000 C CNN
 F 2 "Package_DIP:DIP-16_W7.62mm" H 7850 5550 50  0001 C CNN
 F 3 "https://assets.nexperia.com/documents/data-sheet/74HC_HCT595.pdf" H 7850 5550 50  0001 C CNN
@@
 F 0 "U1" H 2200 658 50  0000 C CNN
 F 1 "MCP1700-3302E_TO92" H 2200 749 50  0000 C CNN
-F 2 "Package_TO_SOT_THT:TO-92_Inline" H 2200 700 50  0001 C CIN
+F 2 "Package_TO_SOT_THT:TO-92_Inline_W4.0mm_Horizontal_FlatSideDown" H 2200 700 50  0001 C CIN
 F 3 "http://ww1.microchip.com/downloads/en/DeviceDoc/20001826D.pdf" H 2200 900 50  0001 C CNN
 	1    2200 900
@@
 F 0 "C3" H 2442 1846 50  0000 L CNN
 F 1 "100n" H 2442 1755 50  0000 L CNN
-F 2 "Capacitor_THT:C_Disc_D3.0mm_W1.6mm_P2.50mm" H 2350 1800 50  0001 C CNN
+F 2 "Capacitor_SMD:C_1206_3216Metric" H 2350 1800 50  0001 C CNN
 F 3 "~" H 2350 1800 50  0001 C CNN
 	1    2350 1800

Commit message: Few small tweaks and add silk
Parts:
- added C4, C5, C6, C7: 100n, Capacitor_SMD:C_1206_3216Metric, symbol Device:C_Small
- added HS1: QR, teatime:__github.com_HarkonenBade_teatime, symbol Mechanical:Heatsink
- R1, R10, R11, R12, R13, R14, R15, R16, R17, R18, R19, R2, R20, R21, R22, R23, R24, R25, R26, R27, R28, R29, R3, R30, R31, R32, R33, R4, R5, R6, R7, R8, R9: footprint Resistor_THT:R_Axial_DIN0204_L3.6mm_D1.6mm_P5.08mm_Horizontal -> Resistor_THT:R_Axial_DIN0204_L3.6mm_D1.6mm_P7.62mm_Horizontal
Connections:
- net +3V3: now also C4.1, C5.1, C6.1, C7.1
- net GND: now also C4.2, C5.2, C6.2, C7.2
Other:
- note added: "74hc595 Decoupling"

Commit message: Switch around various bits: * Add decoupling * Omron button * pth caps
Parts:
- C1, C2: footprint Capacitor_SMD:C_1206_3216Metric -> Capacitor_THT:C_Rect_L4.6mm_W3.0mm_P2.50mm_MKS02_FKP02; Farnell (none) -> 2544872
- C3, C4, C5, C6, C7: footprint Capacitor_SMD:C_1206_3216Metric -> Capacitor_THT:C_Rect_L4.0mm_W2.5mm_P2.50mm; Farnell (none) -> 1141775
- SW1: footprint Button_Switch_THT:SW_PUSH_6mm -> teatime:B3F-40xx
- U6: symbol MCU_Microchip_ATtiny:ATtiny85-20PU -> teatime-rescue:ATtiny85-20PU-MCU_Microchip_ATtiny
Connections:
- net at U2.12 (RCLK), U3.12 (RCLK), U4.12 (RCLK)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: now also U6.5 (AREF/PB0); no longer U6.7 (PB2)
- net at U2.14 (SER): now also U6.7 (PB2); no longer U6.5 (AREF/PB0)
Changed lines of the file:
@@
 F 0 "C1" H 1792 1046 50  0000 L CNN
 F 1 "1u" H 1792 955 50  0000 L CNN
-F 2 "Capacitor_SMD:C_1206_3216Metric" H 1700 1000 50  0001 C CNN
+F 2 "Capacitor_THT:C_Rect_L4.6mm_W3.0mm_P2.50mm_MKS02_FKP02" H 1700 1000 50  0001 C CNN
 F 3 "~" H 1700 1000 50  0001 C CNN
+F 4 "2544872" H 1700 1000 50  0001 C CNN "Farnell"
 	1    1700 1000
-	1    0    0    -1
-$EndComp
-$Comp
-L Device:C_Small C2
-U 1 1 5E46AD91
-P 2700 1000
-F 0 "C2" H 2792 1046 50  0000 L CNN
-F 1 "1u" H 2792 955 50  0000 L CNN
-F 2 "Capacitor_SMD:C_1206_3216Metric" H 2700 1000 50  0001 C CNN
-F 3 "~" H 2700 1000 50  0001 C CNN
-	1    2700 1000
 	1    0    0    -1
 $EndComp
@@
 Connection ~ 2200 1250
 Wire Wire Line
-	2700 900  2500 900
-Wire Wire Line
-	2950 900  2700 900
-Connection ~ 2700 900
-Wire Wire Line
 	1900 900  1700 900
 Connection ~ 1700 900
@@
 $EndComp
 $Comp
-L MCU_Microchip_ATtiny:ATtiny85-20PU U6
+L teatime-rescue:ATtiny85-20PU-MCU_Microchip_ATtiny U6
 U 1 1 5E4A18E1
 P 2700 2600
@@
 F 0 "SW1" V 3654 3448 50  0000 L CNN
 F 1 "SW_Push" V 3745 3448 50  0000 L CNN
-F 2 "Button_Switch_THT:SW_PUSH_6mm" H 3700 3500 50  0001 C CNN
+F 2 "teatime:B3F-40xx" H 3700 3500 50  0001 C CNN
 F 3 "~" H 3700 3500 50  0001 C CNN
 	1    3700 3300
@@
 Connection ~ 3700 3100
 Wire Wire Line
-	4350 2050 4350 2500
-Wire Wire Line
 	3300 2400 4300 2400
-Wire Wire Line
-	3300 2500 4350 2500
-Connection ~ 4350 2500
-Wire Wire Line
-	4350 2500 4350 3250
-Wire Wire Line
-	4250 1550 4250 2300
-Wire Wire Line
-	4250 2300 3300 2300
 $Comp
 L Regulator_Linear:MCP1700-3302E_TO92 U1
@@
 F 0 "C3" H 2442 1846 50  0000 L CNN
 F 1 "100n" H 2442 1755 50  0000 L CNN
-F 2 "Capacitor_SMD:C_1206_3216Metric" H 2350 1800 50  0001 C CNN
+F 2 "Capacitor_THT:C_Rect_L4.0mm_W2.5mm_P2.50mm" H 2350 1800 50  0001 C CNN
 F 3 "~" H 2350 1800 50  0001 C CNN
+F 4 "1141775" H 2350 1800 50  0001 C CNN "Farnell"
 	1    2350 1800
 	1    0    0    -1
@@
 Connection ~ 2700 1700
 $Comp
-L Device:C_Small C4
-U 1 1 5E479313
-P 9050 1300
-F 0 "C4" H 9142 1346 50  0000 L CNN
-F 1 "100n" H 9142 1255 50  0000 L CNN
-F 2 "Capacitor_SMD:C_1206_3216Metric" H 9050 1300 50  0001 C CNN
-F 3 "~" H 9050 1300 50  0001 C CNN
-	1    9050 1300
-	1    0    0    -1
-$EndComp
-$Comp
 L power:GND #PWR020
 U 1 1 5E479439
@@
 $EndComp
 Connection ~ 5450 1350
-$Comp
-L Device:C_Small C5
-U 1 1 5E48E2A0
-P 9400 1300
-F 0 "C5" H 9492 1346 50  0000 L CNN
-F 1 "100n" H 9492 1255 50  0000 L CNN
-F 2 "Capacitor_SMD:C_1206_3216Metric" H 9400 1300 50  0001 C CNN
-F 3 "~" H 9400 1300 50  0001 C CNN
-	1    9400 1300
-	1    0    0    -1
-$EndComp
-$Comp
-L Device:C_Small C6
-U 1 1 5E48E35E
-P 9750 1300
-F 0 "C6" H 9842 1346 50  0000 L CNN
-F 1 "100n" H 9842 1255 50  0000 L CNN
-F 2 "Capacitor_SMD:C_1206_3216Metric" H 9750 1300 50  0001 C CNN
-F 3 "~" H 9750 1300 50  0001 C CNN
-	1    9750 1300
-	1    0    0    -1
-$EndComp
-$Comp
-L Device:C_Small C7
-U 1 1 5E48E422
-P 10100 1300
-F 0 "C7" H 10192 1346 50  0000 L CNN
-F 1 "100n" H 10192 1255 50  0000 L CNN
-F 2 "Capacitor_SMD:C_1206_3216Metric" H 10100 1300 50  0001 C CNN
-F 3 "~" H 10100 1300 50  0001 C CNN
-	1    10100 1300
-	1    0    0    -1
-$EndComp
-Wire Wire Line
-	9050 1400 9400 1400
-Connection ~ 9400 1400
-Wire Wire Line
-	9400 1400 9600 1400
 Connection ~ 9600 1400
-Wire Wire Line
-	9600 1400 9750 1400
-Connection ~ 9750 1400
-Wire Wire Line
-	9750 1400 10100 1400
 $Comp
 L power:+3V3 #PWR019
@@
 	1    0    0    -1
 $EndComp
-Wire Wire Line
-	9050 1200 9400 1200
-Connection ~ 9400 1200
-Wire Wire Line
-	9400 1200 9600 1200
 Connection ~ 9600 1200
-Wire Wire Line
-	9600 1200 9750 1200
-Connection ~ 9750 1200
-Wire Wire Line
-	9750 1200 10100 1200
 Text Notes 9200 1700 0    50   ~ 0
 74hc595 Decoupling
@@
 	1    0    0    -1
 $EndComp
+Wire Wire Line
+	4350 2050 4350 2300
+Connection ~ 4350 2300
+Wire Wire Line
+	4350 2300 4350 3250
+Wire Wire Line
+	3300 2300 4350 2300
+Wire Wire Line
+	4250 1550 4250 2500
+Wire Wire Line
+	4250 2500 3300 2500
+Wire Wire Line
+	9050 1200 9400 1200
+Wire Wire Line
+	9050 1400 9400 1400
+Wire Wire Line
+	9600 1200 9750 1200
+Wire Wire Line
+	9600 1400 9750 1400
+$Comp
+L Device:C_Small C4
+U 1 1 5E494EEA
+P 9050 1300
+F 0 "C4" H 9142 1346 50  0000 L CNN
+F 1 "100n" H 9142 1255 50  0000 L CNN
+F 2 "Capacitor_THT:C_Rect_L4.0mm_W2.5mm_P2.50mm" H 9050 1300 50  0001 C CNN
+F 3 "~" H 9050 1300 50  0001 C CNN
+F 4 "1141775" H 9050 1300 50  0001 C CNN "Farnell"
+	1    9050 1300
+	1    0    0    -1
+$EndComp
+$Comp
+L Device:C_Small C5
+U 1 1 5E495028
+P 9400 1300
+F 0 "C5" H 9492 1346 50  0000 L CNN
+F 1 "100n" H 9492 1255 50  0000 L CNN
+F 2 "Capacitor_THT:C_Rect_L4.0mm_W2.5mm_P2.50mm" H 9400 1300 50  0001 C CNN
+F 3 "~" H 9400 1300 50  0001 C CNN
+F 4 "1141775" H 9400 1300 50  0001 C CNN "Farnell"
+	1    9400 1300
+	1    0    0    -1
+$EndComp
+Connection ~ 9400 1200
+Wire Wire Line
+	9400 1200 9600 1200
+Connection ~ 9400 1400
+Wire Wire Line
+	9400 1400 9600 1400
+$Comp
+L Device:C_Small C6
+U 1 1 5E4950EE
+P 9750 1300
+F 0 "C6" H 9842 1346 50  0000 L CNN
+F 1 "100n" H 9842 1255 50  0000 L CNN
+F 2 "Capacitor_THT:C_Rect_L4.0mm_W2.5mm_P2.50mm" H 9750 1300 50  0001 C CNN
+F 3 "~" H 9750 1300 50  0001 C CNN
+F 4 "1141775" H 9750 1300 50  0001 C CNN "Farnell"
+	1    9750 1300
+	1    0    0    -1
+$EndComp
+Connection ~ 9750 1200
+Wire Wire Line
+	9750 1200 10100 1200
+Connection ~ 9750 1400
+Wire Wire Line
+	9750 1400 10100 1400
+$Comp
+L Device:C_Small C7
+U 1 1 5E4951B6
+P 10100 1300
+F 0 "C7" H 10192 1346 50  0000 L CNN
+F 1 "100n" H 10192 1255 50  0000 L CNN
+F 2 "Capacitor_THT:C_Rect_L4.0mm_W2.5mm_P2.50mm" H 10100 1300 50  0001 C CNN
+F 3 "~" H 10100 1300 50  0001 C CNN
+F 4 "1141775" H 10100 1300 50  0001 C CNN "Farnell"
+	1    10100 1300
+	1    0    0    -1
+$EndComp
+Wire Wire Line
+	2500 900  2700 900
+$Comp
+L Device:C_Small C2
+U 1 1 5E4953EA
+P 2700 1000
+F 0 "C2" H 2792 1046 50  0000 L CNN
+F 1 "1u" H 2792 955 50  0000 L CNN
+F 2 "Capacitor_THT:C_Rect_L4.6mm_W3.0mm_P2.50mm_MKS02_FKP02" H 2700 1000 50  0001 C CNN
+F 3 "~" H 2700 1000 50  0001 C CNN
+F 4 "2544872" H 2700 1000 50  0001 C CNN "Farnell"
+	1    2700 1000
+	1    0    0    -1
+$EndComp
+Connection ~ 2700 900
+Wire Wire Line
+	2700 900  2950 900
+$Comp
+L power:PWR_FLAG #FLG0101
+U 1 1 5E4A085B
+P 700 900
+F 0 "#FLG0101" H 700 975 50  0001 C CNN
+F 1 "PWR_FLAG" H 700 1074 50  0001 C CNN
+F 2 "" H 700 900 50  0001 C CNN
+F 3 "~" H 700 900 50  0001 C CNN
+	1    700  900
+	0    -1   -1   0
+$EndComp
+$Comp
+L power:PWR_FLAG #FLG0102
+U 1 1 5E4A0917
+P 700 1200
+F 0 "#FLG0102" H 700 1275 50  0001 C CNN
+F 1 "PWR_FLAG" V 700 1328 50  0001 L CNN
+F 2 "" H 700 1200 50  0001 C CNN
+F 3 "~" H 700 1200 50  0001 C CNN
+	1    700  1200
+	0    -1   -1   0
+$EndComp
+Connection ~ 700  900
+Connection ~ 700  1200
 $EndSCHEMATC
